File: hardware/kicad_files/tiny_robo_v2/tiny_robo_v2.sch (KiCad schematic (older format))
At the start: 33 parts, among them P1 CONN_8, P2 BATT, P3 CONN_01X02, P4 CONNECTOR, P5 CONNECTOR, P6 CONN_01X02, SW1 SPDT, U1 MCP73831, U2 MIC5265, U3 ESP8266-ESP-03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

Commit message: Changes from loading and unloading kicad project. I have... concerns that this is going to destroy my kicad work.
Parts:
- C1, C2, C3: symbol C -> C-RESCUE-tiny_robo_v2
- C4: symbol CP1 -> CP1-RESCUE-tiny_robo_v2
- Charge1, D2: symbol LED -> LED-RESCUE-tiny_robo_v2
- R1, R10, R11, R12, R13, R2, R3, R4, R5, R6, R7, R8, R9: symbol R -> R-RESCUE-tiny_robo_v2
- SW1: symbol SPDT -> SPDT-RESCUE-tiny_robo_v2
Changed lines of the file:
@@
 EESchema Schematic File Version 2
+LIBS:tiny_robo_v2-rescue
 LIBS:power
 LIBS:device
@@
 LIBS:memory
 LIBS:xilinx
-LIBS:special
 LIBS:microcontrollers
 LIBS:dsp
@@
 LIBS:contrib
 LIBS:valves
-LIBS:shardy
-LIBS:74hct125d
-LIBS:arm-swd-header
-LIBS:esp8266-esp-01
-LIBS:esp8266-esp-03
-LIBS:hm-11
-LIBS:lpc11u14fbd48
-LIBS:mcp1700t-3302e-tt
-LIBS:mcp73831t-2aci-ot
-LIBS:micro_usb_socket
-LIBS:mke02z64vld2
-LIBS:mke04z8vtg4
-LIBS:nrf24l01p_smd
-LIBS:nrf51822-04
-LIBS:nRF24L01+
-LIBS:pp_ws2812b
-LIBS:stm32f37xxx_48pin
-LIBS:stm32f102xx_48pin
-LIBS:stm32f302xx_48pin
-LIBS:switch_china_spdt
-LIBS:uart_pp
-LIBS:usb_plug
-LIBS:open-project
 LIBS:spdt
 LIBS:tiny_robo_v2-cache
@@
 $EndDescr
 $Comp
-L +3.3V #PWR01
+L +3.3V-RESCUE-tiny_robo_v2 #PWR01
 U 1 1 55774122
 P 9250 3400
@@
 Fault1
 $Comp
-L GND #PWR02
+L GND-RESCUE-tiny_robo_v2 #PWR02
 U 1 1 5577082A
 P 6475 1425
@@
 SDA
 $Comp
-L GND #PWR03
+L GND-RESCUE-tiny_robo_v2 #PWR03
 U 1 1 55770098
 P 8050 6850
@@
 $EndComp
 $Comp
-L R R5
+L R-RESCUE-tiny_robo_v2 R5
 U 1 1 5576FFFF
 P 9275 4300
@@
 $EndComp
 $Comp
-L R R8
+L R-RESCUE-tiny_robo_v2 R8
 U 1 1 5576FE5F
 P 10025 5050
@@
 $EndComp
 $Comp
-L R R9
+L R-RESCUE-tiny_robo_v2 R9
 U 1 1 5576FE58
 P 10175 6075
@@
 $EndComp
 $Comp
-L R R7
+L R-RESCUE-tiny_robo_v2 R7
 U 1 1 5576FE2F
 P 9650 4300
@@
 $EndComp
 $Comp
-L R R6
+L R-RESCUE-tiny_robo_v2 R6
 U 1 1 5576FE2B
 P 9450 4300
@@
 $EndComp
 $Comp
-L R R4
+L R-RESCUE-tiny_robo_v2 R4
 U 1 1 5576FE28
 P 7850 6350
@@
 $EndComp
 $Comp
-L R R3
+L R-RESCUE-tiny_robo_v2 R3
 U 1 1 5576FE1B
 P 7650 6350
@@
 $EndComp
 $Comp
-L GND #PWR04
+L GND-RESCUE-tiny_robo_v2 #PWR04
 U 1 1 5575FDC6
 P 4250 4950
@@
 $EndComp
 $Comp
-L +3.3V #PWR05
+L +3.3V-RESCUE-tiny_robo_v2 #PWR05
 U 1 1 5575F5D2
 P 4500 4800
@@
 $EndComp
 $Comp
-L +3.3V #PWR07
+L +3.3V-RESCUE-tiny_robo_v2 #PWR07
 U 1 1 54EFA66A
 P 8550 1325
@@
 $EndComp
 $Comp
-L LED Charge1
+L LED-RESCUE-tiny_robo_v2 Charge1
 U 1 1 54EF9FA6
 P 3650 2050
@@
 $EndComp
 $Comp
-L CP1 C4
+L CP1-RESCUE-tiny_robo_v2 C4
 U 1 1 54EF9F83
 P 8550 1900
@@
 $EndComp
 $Comp
-L R R1
+L R-RESCUE-tiny_robo_v2 R1
 U 1 1 54EF9F5C
 P 4200 2050
@@
 $EndComp
 $Comp
-L R R2
+L R-RESCUE-tiny_robo_v2 R2
 U 1 1 54EF9F56
 P 5400 2300
@@
 $EndComp
 $Comp
-L C C3
+L C-RESCUE-tiny_robo_v2 C3
 U 1 1 54EF9F4F
 P 8225 1900
@@
 $EndComp
 $Comp
-L C C2
+L C-RESCUE-tiny_robo_v2 C2
 U 1 1 54EF9F4A
 P 5650 2250
@@
 $EndComp
 $Comp
-L C C1
+L C-RESCUE-tiny_robo_v2 C1
 U 1 1 54EF9F43
 P 3225 2050
@@
 $EndComp
 $Comp
-L GND #PWR08
+L GND-RESCUE-tiny_robo_v2 #PWR08
 U 1 1 54EF9ED1
 P 4450 2700
@@
 	4500 5100 3650 5100
 $Comp
-L SPDT SW1
+L SPDT-RESCUE-tiny_robo_v2 SW1
 U 1 1 559C6DAD
 P 6400 2000
@@
 	6250 3450 6250 3950
 $Comp
-L GND #PWR09
+L GND-RESCUE-tiny_robo_v2 #PWR09
 U 1 1 559D6D0E
 P 6250 3950
@@
 	6050 5600 6300 5600
 $Comp
-L R R11
+L R-RESCUE-tiny_robo_v2 R11
 U 1 1 566F3103
 P 4575 4325
@@
 $EndComp
 $Comp
-L R R10
+L R-RESCUE-tiny_robo_v2 R10
 U 1 1 566F32C9
 P 4250 4325
@@
 	4250 3975 4250 4075
 $Comp
-L R R12
+L R-RESCUE-tiny_robo_v2 R12
 U 1 1 566F3E82
 P 4850 4350
@@
 	4400 4575 4575 4575
 $Comp
-L R R13
+L R-RESCUE-tiny_robo_v2 R13
 U 1 1 566F47F1
 P 6125 4625
@@
 $EndComp
 $Comp
-L LED D2
+L LED-RESCUE-tiny_robo_v2 D2
 U 1 1 566F4942
 P 5950 4625
