File: hardware/kicad_files/tiny_robo_v2/tiny_robo_v2.kicad_pcb (KiCad board)
At the start: 2 copper layers, 31 parts, among them P1 CONN_01X06, P2 BATT, P3 CONN_01X02, P4 CONNECTOR, P5 CONNECTOR, P6 CONN_01X02, SW1 SPDT, U1 MCP73831, U2 MIC5265, U3 ESP8266-ESP-03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

Commit message: Uploaded new version, buy it at http://dirtypcbs.com/view.php?share=19993&accesskey=05f2c039a03e3f4ff6dc1a4ad2efa9ee
Other:
- board outline added: 25.4 x 39.1 mm
Changed lines of the file:
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@@
     (area 135.353667 84.638999 185.702334 117.4972)
     (thickness 1.6)
-    (drawings 0)
+    (drawings 4)
     (tracks 256)
     (zones 0)
@@
     (pad_to_mask_clearance 0.2)
     (aux_axis_origin 0 0)
-    (visible_elements FFFFFF1F)
+    (visible_elements FFFFFF3F)
     (pcbplotparams
-      (layerselection 0x00030_80000001)
+      (layerselection 0x010f0_80000001)
       (usegerberextensions false)
       (excludeedgelayer true)
@@
       (outputformat 1)
       (mirror false)
-      (drillshape 1)
+      (drillshape 0)
       (scaleselection 1)
       (outputdirectory ""))
@@
     (pad "" thru_hole circle (at 1.50114 0) (size 1.00076 1.00076) (drill 1.00076) (layers *.Cu F.SilkS))
   )
+  (gr_line (start 157.48 114.046) (end 157.48 74.93) (angle 90) (layer Edge.Cuts) (width 0.15))
+  (gr_line (start 182.88 114.046) (end 157.48 114.046) (angle 90) (layer Edge.Cuts) (width 0.15))
+  (gr_line (start 182.88 74.93) (end 182.88 114.046) (angle 90) (layer Edge.Cuts) (width 0.15))
+  (gr_line (start 157.48 74.93) (end 182.88 74.93) (angle 90) (layer Edge.Cuts) (width 0.15))
   (via (at 177.292 103.156) (size 0.6) (drill 0.4) (layers F.Cu B.Cu) (net 1))
   (segment (start 177.292 103.156) (end 177.26 103.124) (width 0.5) (layer B.Cu) (net 1))
